File: Hardware/Basic/Bottom/smart_watch-BASIC-BOTTOM.brd (EAGLE design)
At the start: 38 x 38 mm, 49 parts, among them U2 NRF52832_MODULE_MDBT42, U4 PCF8523

Commit message: Top
Parts:
- added C22: 100n, LinnesLab-Passives:C0603
- added C23, C24: 47p, LinnesLab-Passives:C0603
- added JP2: (no value), LinnesLab-Switches:SMT-JUMPER_2_NO_SILK
- added LED5: RED, LinnesLab-LED:LED-0603
- added LED6: YELLOW, LinnesLab-LED:LED-0603
- added R1, R2: 0, LinnesLab-Passives:R0603
- added R17, R18: 27, LinnesLab-Passives:R0603
- added R19, R20: 1k, LinnesLab-Passives:R0603
- added SW1, SW2: SWITCH.MOM, LinnesLab-Switches:TACTILE_SWITCH_SMD_6.2MM_TALL
- added U5: FT231XS, LinnesLab-DigitalIC:SSOP20_L
- moved R9 39.6 mm to (0.81, -10.5), turned to 0 degrees
- moved R8 37.5 mm to (0.81, -7.82), turned to 0 degrees
- moved LDO2 24.2 mm to (2.92, 22.8)
- moved R15 9.69 mm to (19.7, 12.5)
- moved R11 8.17 mm to (14.1, 6.30)
- moved R12 8.17 mm to (9.12, 6.58)
- moved C6 6.25 mm to (13.6, 2.97)
- moved C21 4.06 mm to (23.3, 12.6)
- moved C5 2.06 mm to (11.6, 2.90)
Connections:
- net VBATT renamed VBAT
- removed net RXD: U2.21
- removed net TXD: U2.19
- new net !CTS: JP2.2, U5.9
- new net FT3V3: U5.13
- new net N$23: R17.2, U5.12
- new net N$24: R18.2, U5.11
- new net N$25: LED5.C, R19.2
- new net N$26: LED6.C, R20.2
- new net RXD.FT: R2.1, U5.4
- new net RXD.NRF: R1.2, U2.21
- new net RXLED: R19.1, U5.17
- new net SW1: SW1.A1
- new net SW2: SW2.A1
- new net TXD.FT: R1.1, U5.20
- new net TXD.NRF: R2.2, U2.19
- new net TXLED: R20.1, U5.10
- net 3.3V: now also C22.2, LED5.A, LED6.A, U5.14, U5.3
- net DTR: now also U5.1
- net GND: now also C22.1, C23.2, C24.1, JP2.1, SW1.B1, SW1.B2, SW2.B1, SW2.B2, U5.16, U5.6
- net SCL: now also R9.1; no longer R8.1
- net SDA: now also R8.1; no longer R9.1
- net USB+: now also C23.1, R18.1
- net USB-: now also C24.2, R17.1
- net V_USB: now also U5.15
