File: Hardware/Basic/Bottom/smart_watch-BASIC-BOTTOM.sch (EAGLE design)
At the start: 49 parts, among them U2 NRF52832_MODULE_MDBT42, U4 PCF8523

Commit message: Top
Parts:
- added C22: 100n, LinnesLab-Passives:CAPACITOR0603
- added C23, C24: 47p, LinnesLab-Passives:CAPACITOR0603
- added JP2: (no value), LinnesLab-Switches:JUMPER-SMT_2_NO_SILK
- added LED5: RED, LinnesLab-LED:LED0603
- added LED6: YELLOW, LinnesLab-LED:LED0603
- added R1, R2: 0, LinnesLab-Passives:RESISTOR0603
- added R17, R18: 27, LinnesLab-Passives:RESISTOR0603
- added R19, R20: 1k, LinnesLab-Passives:RESISTOR0603
- added SW1, SW2: SWITCH.MOM, LinnesLab-Switches:SWITCH.MOM
- added U5: FT231XS, LinnesLab-DigitalIC:FT231XS
Connections:
- removed net RXD: U2.P0.08
- removed net TXD: U2.P0.06
- removed net VBATT: U4.VBAT
- new net !CTS: JP2.2, U5.!CTS
- new net FT3V3: U5.3V3OUT
- new net N$23: R17.2, U5.USBDM
- new net N$24: R18.2, U5.USBDP
- new net N$25: LED5.C, R19.2
- new net N$26: LED6.C, R20.2
- new net RXD.FT: R2.1, U5.RXD
- new net RXD.NRF: R1.2, U2.P0.08
- new net RXLED: R19.1, U5.CBUS1
- new net SW1: SW1.1
- new net SW2: SW2.1
- new net TXD.FT: R1.1, U5.TXD
- new net TXD.NRF: R2.2, U2.P0.06
- new net TXLED: R20.1, U5.CBUS2
- net 3.3V: now also C22.2, LED5.A, LED6.A, U5.!RESET, U5.VCCIO
- net DTR: now also U5.!DTR
- net GND: now also C22.1, C23.2, C24.1, JP2.1, SW1.3, SW1.4, SW2.3, SW2.4, U5.GND@16, U5.GND@6
- net SCL: now also R9.1; no longer R8.1
- net SDA: now also R8.1; no longer R9.1
- net USB+: now also C23.1, R18.1
- net USB-: now also C24.2, R17.1
- net V_USB: now also U5.VCC
Other:
- note added: "Bottons"
- note added: "I don't remember if CTS needs to be grounded or left floating so here's a jumper to ground so it can be configued either way dynamically."
- note added: "TXD goes to RX on the other device RXD goes to TX on the other device"
- note added: "USB to Serial"
- note removed: "Buttons"
- moved on the sheet: C14, C20, C21, C5, C6, CHRG2, CORTEX1, D1, D4, D5, J2, LDO2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
